File: nimh-charger.kicad_sch (KiCad schematic)
At the start: 8 parts

Commit message: Assign PCB layouts.
Parts:
- added BT? (x3): Battery_Cell, symbol Device:Battery_Cell
- added D? (x3): RED LED, LED_SMD:LED_1206_3216Metric_Pad1.42x1.75mm_HandSolder, symbol Device:LED
- added D? (x3): 1N4007, Diode_SMD:D_SOD-123F, symbol Diode:1N4007
- added R? (x6): 220R, Resistor_SMD:R_1206_3216Metric_Pad1.30x1.75mm_HandSolder, symbol Device:R
- BT1: value (none) -> Battery_Cell
- D3: value LED -> (none)
- R1: value (none) -> 470R; footprint (none) -> Resistor_SMD:R_1206_3216Metric_Pad1.30x1.75mm_HandSolder
- R2, R3: value (none) -> 220R; footprint (none) -> Resistor_SMD:R_1206_3216Metric_Pad1.30x1.75mm_HandSolder
Connections:
- net +5V: now also D?.2 (A), D?.2 (A), D?.2 (A)
- net GND: now also BT?.2 (-), BT?.2 (-), BT?.2 (-); no longer J1.6 (Shield)
- new net: D?.1 (K), R?.1 (x3)
- new net: BT?.1 (+), R?.2, R?.2 (x3)
- new net: D?.1 (K), D?.2 (A), R?.1 (x3)
- no-connect marks 3 -> 4
Other:
- note added: "Charger Bank"
- note added: "MicroUSB Power Supply"
- note added: "NIMH trickle-charging must remain below 0.05C (i.e. <40mA for 800mAh cell). Therefore, resistors calculated to provide max 20mA current to each cell at end of charge: Current = [[5.0V USB - 0.6V diode - 1.35V cell] + [5V - 0.6V - 1.35V - 2V LED]] / 220R = 19mA"
- note added: "Power Indicator"
- moved on the sheet: BT1, D1, D2, D3, J1, R1, R2, R3

Commit message: Create and assign cell holder layout.
Parts:
- BT1: value Battery_Cell -> (none)
- BT2: renamed from BT?; value Battery_Cell -> (none)
- D1: renamed from D2; value (none) -> 1N4007; footprint (none) -> Diode_SMD:D_SOD-123F
- D5: renamed from D3; value (none) -> RED LED; footprint (none) -> LED_SMD:LED_1206_3216Metric_Pad1.42x1.75mm_HandSolder
- D9: renamed from D1; value (none) -> GREEN LED; footprint (none) -> LED_SMD:LED_1206_3216Metric_Pad1.42x1.75mm_HandSolder
- J1: value (none) -> USB_B_Micro; footprint (none) -> Connector_USB:USB_Micro-B_Amphenol_10118194_Horizontal
- gave numbers to parts that had none: 14
- renumbered R2 to R1, R3 to R2, R1 to R9
