File: nimh-charger.kicad_pcb (KiCad board)
At the start: 2 copper layers, 70 x 75 mm, 23 parts, among them J1 USB_B_Micro

Commit message: Generate plots.
Other:
- board text added: "NiMH Charger Rev 1-0 Alexander Fraser 12 July 2022"
